Commit message: 二刷到机器人建模和仿真

File: src/fishbot_description/urdf/fishbot/actuator/caster.urdf.xacro (robot description, xacro)
@@ -2,5 +2,5 @@
 <robot xmlns:xacro="http://www.ros.org/wiki/xacro">
     <xacro:include filename="$(find fishbot_description)/urdf/fishbot/common_inertia.xacro"/>
-    <!--    机器人的IMU部件，惯性测量传感器-->
+    <!--    机器人的万相轮-->
     <xacro:macro name="caster_xacro" params="caster_name xyz">
         <gazebo reference="${caster_name}_link">

File: src/fishbot_description/urdf/fishbot/actuator/wheel.urdf.xacro (robot description, xacro)
@@ -2,5 +2,5 @@
 <robot xmlns:xacro="http://www.ros.org/wiki/xacro">
     <xacro:include filename="$(find fishbot_description)/urdf/fishbot/common_inertia.xacro"/>
-    <!--    机器人的IMU部件，惯性测量传感器-->
+    <!--    机器人的动力轮-->
     <xacro:macro name="wheel_xacro" params="wheel_name xyz">
         <gazebo reference="${wheel_name}_link">

File: src/fishbot_description/urdf/fishbot/base.urdf.xacro (robot description, xacro)
@@ -5,4 +5,7 @@
     <!--    机器人的身体部分-->
     <xacro:macro name="base_xacro" params="length radius">
+        <gazebo reference="base_link">
+            <material>Gazebo/White</material>
+        </gazebo>
         <link name="base_link">
             <!-- 部件的外观描述-->

File: src/fishbot_description/urdf/fishbot/common_inertia.xacro (robot description, xacro)
@@ -1,4 +1,4 @@
 <?xml version="1.0"?>
-<!--惯性质量-->
+<!--惯性质量 可以在http://fishros.org/doc/nav2/setup_guides/urdf/setup_urdf.html找到-->
 <robot xmlns:xacro="http://www.ros.org/wiki/xacro">
     <xacro:macro name="box_inertia" params="m w h d">

File: src/fishbot_description/urdf/fishbot/plugins/gazebo_control_plugin.xacro (robot description, xacro)
@@ -6,7 +6,10 @@
                 <ros>
                     <namespace>/</namespace>
+                    <!--                    订阅话题名-->
                     <remapping>cmd_vel:=cmd_vel</remapping>
+                    <!--                    发布话题名-->
                     <remapping>odom:=odom</remapping>
                 </ros>
+                <!--                发布频率-->
                 <update_rate>30</update_rate>
                 <!-- wheels -->

File: src/fishbot_description/urdf/fishbot/plugins/gazebo_sensor_plugin.xacro (robot description, xacro)
@@ -9,5 +9,7 @@
                         <remapping>~/out:=scan</remapping>
                     </ros>
+                    <!--                    数据类型-->
                     <output_type>sensor_msgs/LaserScan</output_type>
+                    <!--                    数据中坐标系-->
                     <frame_name>laser_link</frame_name>
                 </plugin>
@@ -126,4 +128,5 @@
                 </image>
                 <distortion>
+                    <!--                    通过标定得到的相机的畸变参数-->
                     <k1>0.0</k1>
                     <k2>0.0</k2>

File: src/fishbot_description/urdf/fishbot/sensor/camera.urdf.xacro (robot description, xacro)
@@ -19,5 +19,5 @@
                 </material>
             </visual>
-<!--            碰撞属性-->
+            <!--            碰撞属性-->
             <collision>
                 <!-- 沿着自己几何中心的偏移和旋转-->
@@ -33,11 +33,13 @@
                 </material>
             </collision>
-            <xacro:box_inertia m="0.01" w="0.02" h="0.10" d="0.02" />
+            <xacro:box_inertia m="0.01" w="0.02" h="0.10" d="0.02"/>
         </link>
+        <!--        虚拟部件，用于修正相机坐标系-->
         <link name="${camera_name}_optical_link"></link>
         <joint name="${camera_name}_optical_joint" type="fixed">
-            <parent link="${camera_name}_link" />
-            <child link="${camera_name}_optical_link" />
-            <origin xyz="0 0 0" rpy="${-pi/2} 0 ${-pi/2}" />
+            <parent link="${camera_name}_link"/>
+            <child link="${camera_name}_optical_link"/>
+            <!--            右手坐标系，将相机的旋转到，X轴正向和base_link的右一个方向，Y轴正向和base_link的下一个方向，Z轴和base_link的X轴一个方向-->
+            <origin xyz="0 0 0" rpy="${-pi/2} 0 ${-pi/2}"/>
         </joint>
         <!--    机器人的关节，用来组合机器人的部件-->

File: src/fishbot_description/urdf/fishbot/sensor/laser.urdf.xacro (robot description, xacro)
@@ -2,5 +2,5 @@
 <robot xmlns:xacro="http://www.ros.org/wiki/xacro">
     <xacro:include filename="$(find fishbot_description)/urdf/fishbot/common_inertia.xacro"/>
-    <!--    机器人的IMU部件，惯性测量传感器-->
+    <!--    机器人的激光雷达-->
     <xacro:macro name="laser_xacro" params="laser_name xyz">
         <!--        gazebo扩展-->
